File: BlueBikes/battery_charger/battery_charger.kicad_sch (KiCad schematic)
At the start: 6 parts, among them J1 Barrel_Jack, J2 Conn_01x02, U1 LM317_TO-220

Commit message: update various PCB
Parts:
- added C1: 0.1uF, symbol Device:C
Connections:
- net GND: now also C1.2
- net at J1.1, U1.3 (VI): now also C1.1
Other:
- note added: "(optional, prevent possible oscillation)"
Changed lines of the file:
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@@
 	(paper "A")
+	(junction
+		(at 58.42 78.74)
+		(diameter 0)
+		(color 0 0 0 0)
+	)
 	(junction
 		(at 99.06 76.2)
@@
 		(color 0 0 0 0)
 	)
+	(junction
+		(at 66.04 59.69)
+		(diameter 0)
+		(color 0 0 0 0)
+	)
 	(wire
 		(pts
@@
 	(wire
 		(pts
+			(xy 66.04 59.69) (xy 66.04 67.31)
+		)
+		(stroke
+			(width 0)
+			(type default)
+		)
+	)
+	(wire
+		(pts
 			(xy 114.3 62.23) (xy 111.76 62.23)
 		)
@@
 	(wire
 		(pts
+			(xy 66.04 78.74) (xy 58.42 78.74)
+		)
+		(stroke
+			(width 0)
+			(type default)
+		)
+	)
+	(wire
+		(pts
 			(xy 99.06 76.2) (xy 99.06 77.47)
 		)
@@
 	(wire
 		(pts
+			(xy 58.42 78.74) (xy 58.42 83.82)
+		)
+		(stroke
+			(width 0)
+			(type default)
+		)
+	)
+	(wire
+		(pts
+			(xy 66.04 74.93) (xy 66.04 78.74)
+		)
+		(stroke
+			(width 0)
+			(type default)
+		)
+	)
+	(wire
+		(pts
 			(xy 77.47 67.31) (xy 77.47 76.2)
 		)
@@
 	(wire
 		(pts
-			(xy 58.42 64.77) (xy 58.42 67.31)
+			(xy 58.42 64.77) (xy 58.42 78.74)
 		)
 		(stroke
@@
 	(wire
 		(pts
-			(xy 55.88 59.69) (xy 69.85 59.69)
+			(xy 55.88 59.69) (xy 66.04 59.69)
 		)
 		(stroke
@@
 		(pts
 			(xy 85.09 59.69) (xy 88.9 59.69)
+		)
+		(stroke
+			(width 0)
+			(type default)
+		)
+	)
+	(wire
+		(pts
+			(xy 66.04 59.69) (xy 69.85 59.69)
 		)
 		(stroke
@@
 			)
 			(justify left)
+		)
+	)
+	(text "(optional, prevent\npossible oscillation)"
+		(exclude_from_sim no)
+		(at 73.406 81.534 0)
+		(effects
+			(font
+				(size 1.27 1.27)
+			)
 		)
 	)
@@
 	)
 	(symbol
+		(lib_id "Device:C")
+		(at 66.04 71.12 0)
+		(unit 1)
+		(exclude_from_sim no)
+		(in_bom yes)
+		(on_board yes)
+		(dnp no)
+		(fields_autoplaced yes)
+		(property "Reference" "C1"
+			(at 69.85 69.8499 0)
+			(effects
+				(font
+					(size 1.27 1.27)
+				)
+				(justify left)
+			)
+		)
+		(property "Value" "0.1uF"
+			(at 69.85 72.3899 0)
+			(effects
+				(font
+					(size 1.27 1.27)
+				)
+				(justify left)
+			)
+		)
+		(property "Footprint" ""
+			(at 67.0052 74.93 0)
+			(effects
+				(font
+					(size 1.27 1.27)
+				)
+				(hide yes)
+			)
+		)
+		(property "Datasheet" "~"
+			(at 66.04 71.12 0)
+			(effects
+				(font
+					(size 1.27 1.27)
+				)
+				(hide yes)
+			)
+		)
+		(property "Description" "Unpolarized capacitor"
+			(at 66.04 71.12 0)
+			(effects
+				(font
+					(size 1.27 1.27)
+				)
+				(hide yes)
+			)
+		)
+		(pin "2"
+		)
+		(pin "1"
+		)
+		(instances
+			(project ""
+				(path "/b2c0b0b2-7b71-486f-a02b-8f7414a6e628"
+					(reference "C1")
+					(unit 1)
+				)
+			)
+		)
+	)
+	(symbol
 		(lib_id "Connector:Barrel_Jack")
 		(at 48.26 62.23 0)
@@
 	(symbol
 		(lib_id "power:GND")
-		(at 58.42 67.31 0)
+		(at 58.42 83.82 0)
 		(unit 1)
 		(exclude_from_sim no)
@@
 		(fields_autoplaced yes)
 		(property "Reference" "#PWR02"
-			(at 58.42 73.66 0)
+			(at 58.42 90.17 0)
 			(effects
 				(font
@@
 		)
 		(property "Value" "GND"
-			(at 58.42 72.39 0)
+			(at 58.42 88.9 0)
 			(effects
 				(font
@@
 		)
 		(property "Footprint" ""
-			(at 58.42 67.31 0)
+			(at 58.42 83.82 0)
 			(effects
 				(font
@@
 		)
 		(property "Datasheet" ""
-			(at 58.42 67.31 0)
+			(at 58.42 83.82 0)
 			(effects
 				(font
@@
 		)
 		(property "Description" "Power symbol creates a global label with name \"GND\" , ground"
-			(at 58.42 67.31 0)
-			(effects
-				(font
+			(at 58.42 83.82 0)
+			(effects
+				(font
